File: 01_DESIGN/Project_VD/Project_VD.kicad_pcb (KiCad board)
At the start: 4 copper layers, 100 x 100 mm, 108 parts, among them J1 12V, J2 USB_B_Micro, J3 JTAG, J4 NTC1, J5 JTAG, U1 LM1117MP-3.3, U2 LM2596S-5, U3 STM32H745ZIT3, U4 MTFC32GAZAQDW-AAT, U5 ISO7721DR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

Commit message: update 21/06/2026
Parts:
- added NT1: NetTie_2, NetTie:NetTie-2_SMD_Pad0.5mm, F.Cu at (203.5, 108.1)
- added NT2: NetTie_2, NetTie:NetTie-2_SMD_Pad0.5mm, F.Cu at (276.5, 107.4)
- added NT3: NetTie_2, NetTie:NetTie-2_SMD_Pad0.5mm, F.Cu at (203.5, 192.6)
- added NT4: NetTie_2, NetTie:NetTie-2_SMD_Pad0.5mm, F.Cu at (296.5, 191.9)
- moved H2 253.1 mm to (292.6, 192.6)
- moved H1 198.5 mm to (272.6, 107.4)
- moved H3 184.9 mm to (207.4, 192.6)
- moved H4 130.2 mm to (207.4, 107.4)
- moved L2 32.7 mm to (131.5, 114.0)
- moved C10 32.7 mm to (94.4, 62.7)
- moved C11 32.7 mm to (94.4, 65.2)
- moved C12 32.7 mm to (94.4, 67.7)
- moved C2 32.7 mm to (148.5, 68.9)
- moved C21 32.7 mm to (102.4, 50.2)
- moved C22 32.7 mm to (102.4, 52.7)
- moved C23 32.7 mm to (102.4, 55.2)
- moved C24 32.7 mm to (102.4, 57.7)
- moved C25 32.7 mm to (102.4, 60.2)
- moved C26 32.7 mm to (102.4, 62.7)
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Connections:
- H1 pad 1: GND -> /POWER 12 - 5V & 5 - 3.3V/SHIELDING
- H2 pad 1: GND -> /POWER 12 - 5V & 5 - 3.3V/SHIELDING
- H3 pad 1: GND -> /POWER 12 - 5V & 5 - 3.3V/SHIELDING
- H4 pad 1: GND -> /POWER 12 - 5V & 5 - 3.3V/SHIELDING
Routing:
- net /POWER 12 - 5V & 5 - 3.3V/SHIELDING: track 0.00 -> 1539.4 mm, vias 0 -> 252
Other:
- outline, holes or cut-outs redrawn
