File: 01_DESIGN/Project_VD/Project_VD.kicad_pcb (KiCad board)
At the start: 4 copper layers, 100 x 100 mm, 112 parts, among them J1 12V, J2 USB_B_Micro, J3 JTAG, J4 NTC1, J5 JTAG, U1 LM1117MP-3.3, U2 LM2596S-5, U3 STM32H745ZIT3, U4 MTFC32GAZAQDW-AAT, U5 ISO7721DR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

Commit message: update Layout PCB
Parts:
- moved L2 4.06 mm to (266.4, 121.1), turned to 90 degrees
- moved C63 3.50 mm to (264.7, 121.4), turned to 90 degrees
- moved C64 3.50 mm to (268.1, 121.4), turned to -90 degrees
- moved C57 0.80 mm to (254.9, 114.3)
Routing:
- net /MCU ATMEGA324PA/AVR_JTAG_nRESET: track 32.3 -> 48.6 mm
- net /eMMC2/eMMC_SDMMC2_D2: track 43.3 -> 54.9 mm
- net /eMMC2/eMMC_SDMMC2_D3: track 45.6 -> 53.5 mm
- net /MCU ATMEGA324PA/AVR_JTAG_TCK: track 20.7 -> 27.8 mm
- net /eMMC2/eMMC_SDMMC2_CMD: track 45.0 -> 51.2 mm
- net /eMMC2/eMMC_SDMMC2_CK: track 44.7 -> 49.3 mm
- net /eMMC2/eMMC_SDMMC2_D0: track 54.3 -> 55.9 mm
- net /eMMC2/eMMC_SDMMC2_D1: track 45.9 -> 47.5 mm
- net /MCU ATMEGA324PA/AVR_JTAG_TDO: track 17.5 -> 18.5 mm
Other:
- outline, holes or cut-outs redrawn
