File: 01_DESIGN/Project_VD/Project_VD.kicad_pcb (KiCad board)
At the start: 4 copper layers, 100 x 100 mm, 112 parts, among them J1 12V, J2 USB_B_Micro, J3 JTAG, J4 NTC1, J5 JTAG, U1 LM1117MP-3.3, U2 LM2596S-5, U3 STM32H745ZIT3, U4 MTFC32GAZAQDW-AAT, U5 ISO7721DR, U6 OPA2340, U7 ATMEGA324PA, Y1 25MHz, Y2 8MHz

Commit message: hoan thanh Task 1
Other:
- board text added: "+12V GND"
