File: 01_DESIGN/Project_VD/_restore_backup_2026-06-25T11-07-44-690/POWER SUPPLY.kicad_sch (KiCad schematic)
At the start: 26 parts, among them J1 12V, J2 USB_B_Micro, U1 LM1117MP-3.3, U2 LM2596S-5

Commit message: update Layout PCB
Parts:
- C1: MANUFACTURER (none) -> Panasonic; Manufacturer Panasonic -> (none)
Changed lines of the file:
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@@
 			)
 		)
-		(property "Manufacturer" "Panasonic"
+		(property "MANUFACTURER" "Panasonic"
 			(at 55.88 33.02 0)
 			(hide yes)
