File: 01_DESIGN/Project_VD/_restore_backup_2026-06-25T11-07-44-690/Project_VD.kicad_pcb (KiCad board)
At the start: 4 copper layers, 100 x 100 mm, 112 parts, among them J1 12V, J2 USB_B_Micro, J3 JTAG, J4 NTC1, J5 JTAG, U1 LM1117MP-3.3, U2 LM2596S-5, U3 STM32H745ZIT3, U4 MTFC32GAZAQDW-AAT, U5 ISO7721DR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

Commit message: update Layout PCB
Routing:
- net /MCU STM32H745ZIT3/VBAT: track 22.3 -> 3.32 mm, vias 2 -> 0
- net GND: track 172.5 -> 169.0 mm, vias 110 -> 109
- net +3.3V: track 136.7 -> 135.7 mm, vias 50 -> 49
- net /MCU ATMEGA324PA/ADC_TEMP1: track 14.9 -> 14.1 mm
- net +5V: track 41.5 -> 40.9 mm, vias 14 -> 13
Changed lines of the file:
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@@
 		(capping no)
 		(filling no)
-		(zone_defaults)
 		(pcbplotparams
 			(layerselection 0x00000000_00000000_55555555_5755f5ff)
@@
 		(tags "LED")
 		(property "Reference" "D3"
-			(at 0 -1.5 0)
+			(at 0 -1.43 0)
 			(layer "F.SilkS")
 			(effects
@@
 		(tags "capacitor")
 		(property "Reference" "C4"
-			(at 0.175 -1.8 180)
+			(at 0.775 -1.8 180)
 			(layer "F.SilkS")
 			(effects
@@
 		(descr "SMD3225/4, Crystal, 3.2x2.5mm package, SMD, http://www.txccrystal.com/images/pdf/7m-accuracy.pdf")
 		(property "Reference" "Y2"
-			(at -2.8 1.1 180)
+			(at -2.7 1.1 180)
 			(layer "F.SilkS")
 			(effects
@@
 		(tags "LQFP QFP Microchip_144-Lead-Plastic-Low-Profile-Quad-Flatpack-(PL) Microsemi_TQ144")
 		(property "Reference" "U3"
-			(at -12.1375 -9.8 0)
+			(at -12.1 -9.8 0)
 			(layer "F.SilkS")
 			(effects
@@
 		(tags "capacitor electrolytic")
 		(property "Reference" "C2"
-			(at -5.55 -4 0)
+			(at 0 -5.2 0)
 			(layer "F.SilkS")
 			(effects
@@
 		(tags "LED")
 		(property "Reference" "D2"
-			(at 0 -1.5 0)
+			(at 0 -1.43 0)
 			(layer "F.SilkS")
 			(effects
@@
 		(tags "capacitor")
 		(property "Reference" "C48"
-			(at 0 -3.2 0)
+			(at 0 -3.7 0)
 			(layer "B.SilkS")
 			(effects
@@
 		(tags "capacitor")
 		(property "Reference" "C47"
-			(at 0 -3.3 0)
+			(at 0 -4.2 0)
 			(layer "B.SilkS")
 			(effects
@@
 	)
 	(gr_rect
-		(start 230.5 189.6)
-		(end 233.7 197.3)
+		(start 230.6 189.7)
+		(end 233.6 197.2)
 		(stroke
 			(width 0.1)
@@
 	)
 	(segment
-		(start 246.7 122.6)
-		(end 246.7 123.2)
-		(width 0.5)
-		(layer "F.Cu")
-		(net "+5V")
-	)
-	(segment
 		(start 247.34 110.24)
 		(end 247.2 110.1)
@@
 	)
 	(via
-		(at 246.7 123.2)
-		(size 0.6)
-		(drill 0.3)
-		(layers "F.Cu" "B.Cu")
-		(net "+5V")
-	)
-	(via
 		(at 252.5 135)
 		(size 0.4)
@@
 	)
 	(segment
-		(start 276.223756 194.65)
-		(end 276.223756 192.323756)
-		(width 1)
-		(layer "F.Cu")
-		(net "GND")
-	)
-	(segment
 		(start 243.3 127.475)
 		(end 243.3 127.7)
@@
 	)
 	(via
-		(at 227.95 186.9)
+		(at 227.95 188.15)
 		(size 0.4)
 		(drill 0.2)
@@
 		(net "GND")
 	)
-	(via
-		(at 276.223756 192.323756)
-		(size 0.6)
-		(drill 0.3)
-		(layers "F.Cu" "B.Cu")
-		(net "GND")
-	)
 	(segment
 		(start 232.9 182.2)
@@
 	)
 	(segment
-		(start 227.95 189.5)
-		(end 227.95 186.9)
-		(width 0.3)
-		(layer "B.Cu")
-		(net "GND")
-	)
-	(segment
 		(start 222.95 188.9)
 		(end 222.95 189.5)
@@
 	)
 	(segment
-		(start 227.95 187.5)
-		(end 227.95 186.9)
-		(width 0.3)
-		(layer "B.Cu")
-		(net "GND")
-	)
-	(segment
 		(start 227.45 192.575)
 		(end 228.4 192.575)
@@
 	)
 	(segment
+		(start 227.95 189.5)
+		(end 227.95 188.15)
+		(width 0.3)
+		(layer "B.Cu")
+		(net "GND")
+	)
+	(segment
+		(start 227.95 187.5)
+		(end 227.95 188.15)
+		(width 0.3)
+		(layer "B.Cu")
+		(net "GND")
+	)
+	(segment
 		(start 222.95 182)
 		(end 222.95 182.5)
@@
 	)
 	(segment
-		(start 264.15 151.525)
-		(end 264.15 150.5)
-		(width 0.3)
-		(layer "F.Cu")
-		(net "+3.3V")
-	)
-	(segment
 		(start 258.1625 148.575)
 		(end 259.7625 148.575)
@@
 		(net "+3.3V")
 	)
-	(via
-		(at 264.15 150.5)
-		(size 0.6)
-		(drill 0.3)
-		(layers "F.Cu" "B.Cu")
-		(net "+3.3V")
-	)
 	(segment
 		(start 224.5 182.5)
@@
 	)
 	(segment
-		(start 232.58 184.93)
-		(end 231.83 184.93)
-		(width 0.3)
-		(layer "F.Cu")
-		(net "Net-(U4C-VDDIM)")
-	)
-	(segment
-		(start 231.83 184.93)
-		(end 231.4 184.5)
+		(start 238.3 184.6)
+		(end 237.6 185.3)
 		(width 0.3)
 		(layer "F.Cu")
@@
 	)
 	(segment
-		(start 232.81 184.7)
-		(end 232.58 184.93)
+		(start 237.6 185.3)
+		(end 232.95 185.3)
 		(width 0.3)
 		(layer "F.Cu")
@@
 	)
 	(segment
-		(start 233.5 184.7)
-		(end 232.81 184.7)
+		(start 231.4 184.5)
+		(end 231.83 184.93)
 		(width 0.3)
 		(layer "F.Cu")
@@
 	)
 	(segment
-		(start 234.1 185.3)
-		(end 237.6 185.3)
+		(start 232.95 185.3)
+		(end 232.9 185.25)
 		(width 0.3)
 		(layer "F.Cu")
@@
 	)
 	(segment
-		(start 237.6 185.3)
-		(end 238.3 184.6)
+		(start 232.58 184.93)
+		(end 232.9 185.25)
 		(width 0.3)
 		(layer "F.Cu")
@@
 	)
 	(segment
-		(start 233.5 184.7)
-		(end 234.1 185.3)
+		(start 231.83 184.93)
+		(end 232.58 184.93)
 		(width 0.3)
 		(layer "F.Cu")
@@
 	)
 	(via
-		(at 233.5 184.7)
+		(at 232.9 185.25)
 		(size 0.4)
 		(drill 0.2)
@@
 	)
 	(segment
-		(start 233.475 184.675)
-		(end 233.5 184.7)
-		(width 0.3)
-		(layer "B.Cu")
-		(net "Net-(U4C-VDDIM)")
-	)
-	(segment
 		(start 232.9 184.675)
-		(end 233.475 184.675)
+		(end 232.9 185.25)
 		(width 0.3)
 		(layer "B.Cu")
@@
 	)
 	(segment
-		(start 260.6 164.5)
-		(end 260.2 164.5)
-		(width 0.3)
-		(layer "F.Cu")
-		(net "/MCU STM32H745ZIT3/VBAT")
-	)
-	(segment
-		(start 276.2 165.326244)
-		(end 276.223756 165.35)
-		(width 1)
-		(layer "F.Cu")
-		(net "/MCU STM32H745ZIT3/VBAT")
-	)
-	(segment
-		(start 260.9 164.8)
-		(end 260.6 164.5)
-		(width 0.3)
-		(layer "F.Cu")
-		(net "/MCU STM32H745ZIT3/VBAT")
-	)
-	(segment
-		(start 276.2 163.752488)
-		(end 276.2 165.326244)
-		(width 1)
-		(layer "F.Cu")
-		(net "/MCU STM32H745ZIT3/VBAT")
-	)
-	(segment
 		(start 257.725 165.15)
 		(end 260.55 165.15)
@@
 		(net "/MCU STM32H745ZIT3/VBAT")
 	)
-	(via
-		(at 276.2 163.752488)
-		(size 0.6)
-		(drill 0.3)
-		(layers "F.Cu" "B.Cu")
-		(net "/MCU STM32H745ZIT3/VBAT")
-	)
-	(via
-		(at 260.2 164.5)
-		(size 0.6)
-		(drill 0.3)
-		(layers "F.Cu" "B.Cu")
-		(net "/MCU STM32H745ZIT3/VBAT")
-	)
-	(segment
-		(start 260.45 164.75)
-		(end 275.202488 164.75)
-		(width 1)
-		(layer "B.Cu")
-		(net "/MCU STM32H745ZIT3/VBAT")
-	)
-	(segment
-		(start 275.202488 164.75)
-		(end 276.2 163.752488)
-		(width 1)
-		(layer "B.Cu")
-		(net "/MCU STM32H745ZIT3/VBAT")
-	)
-	(segment
-		(start 260.2 164.5)
-		(end 260.45 164.75)
-		(width 1)
-		(layer "B.Cu")
-		(net "/MCU STM32H745ZIT3/VBAT")
-	)
 	(segment
 		(start 258.2 117.5375)
@@
 	)
 	(segment
-		(start 259 117.5375)
-		(end 259.8 117.5375)
-		(width 0.32)
-		(layer "F.Cu")
-		(net "/MCU ATMEGA324PA/ADC_TEMP1")
-	)
-	(segment
 		(start 261.4625 120.8)
 		(end 261.4625 121.6)
@@
 	)
 	(segment
-		(start 248.885 151.65)
-		(end 273.31 151.65)
+		(start 261.765 165.735)
+		(end 274.3 153.2)
 		(width 0.3)
 		(layer "B.Cu")
@@
 	)
 	(segment
-		(start 273.31 151.65)
+		(start 274.3 153.2)
 		(end 274.3 152.64)
 		(width 0.3)
@@
 	(segment
 		(start 234.8 165.735)
-		(end 248.885 151.65)
+		(end 261.765 165.735)
 		(width 0.3)
 		(layer "B.Cu")
